Commit message: Added collision objects for robot table

File: process_visualizer/urdf/robot_table.urdf (robot description, URDF)
Before this commit: robot robot_table, 2 links, 1 joints
Links:
- link robot_table_origin: geometry visual mesh filename=package://process_visualizer/resources/table.stl scale=1 1 1

File: universal_robot/ur_description/urdf/ur5_robot.urdf.xacro (robot description, xacro)
@@ -2,4 +2,6 @@
 <robot xmlns:xacro="http://wiki.ros.org/xacro"
        name="ur5" >
+  <xacro:arg name="rob_xyz" default="0.0 0.0 0.0"/>
+  <xacro:arg name="rob_rpy" default="0.0 0.0 0.0"/>
   <xacro:arg name="transmission_hw_interface" default="hardware_interface/PositionJointInterface"/>
   <!-- common stuff -->
@@ -15,5 +17,5 @@
     <parent link="world" />
     <child link = "base_link" />
-    <origin xyz="0.0 0.0 0.0" rpy="0.0 0.0 0.0" />
+    <origin xyz="$(arg rob_xyz)" rpy="$(arg rob_rpy)" />
   </joint>
 </robot>
