Commit message: Added milling robot ur10

File: universal_robot/ur_description/urdf/ur10.urdf.xacro (robot description, xacro)
@@ -312,4 +312,5 @@
         <geometry>
           <box size="0.01 0.01 0.01"/>
+          <!-- <mesh filename="package://process_visualizer/resources/milling_tool.stl"/> -->
         </geometry>
         <origin rpy="0 0 0" xyz="-0.01 0 0"/>
@@ -330,5 +331,20 @@
     </joint>
     <!-- Frame coincident with all-zeros TCP on UR controller -->
-    <link name="${prefix}tool0"/>
+    <link name="${prefix}tool0">
+      <collision>
+        <geometry>
+          <!-- <box size="0.01 0.01 0.01"/> -->
+          <mesh filename="package://process_visualizer/resources/milling_tool.stl"/>
+        </geometry>
+      </collision>
+        <visual>
+        <geometry>
+          <!-- <box size="0.01 0.01 0.01"/> -->
+          <mesh filename="package://process_visualizer/resources/milling_tool.stl"/>
+        </geometry>
+        </visual>
+        <origin rpy="0 0 0" xyz="0 0 0"/>
+      <!-- </collision> -->
+    </link>
     <joint name="${prefix}wrist_3_link-tool0_fixed_joint" type="fixed">
       <origin xyz="0 ${wrist_3_length} 0" rpy="${pi/-2.0} 0 0"/>

File: universal_robot/ur_description/urdf/ur10_robot.urdf.xacro (robot description, xacro)
@@ -2,4 +2,6 @@
 <robot xmlns:xacro="http://wiki.ros.org/xacro"
        name="ur10" >
+  <xacro:arg name="rob_xyz" default="0.0 0.0 0.0"/>
+  <xacro:arg name="rob_rpy" default="0.0 0.0 0.0"/>
   <xacro:arg name="transmission_hw_interface" default="hardware_interface/PositionJointInterface"/>
   <!-- common stuff -->
@@ -15,5 +17,5 @@
     <parent link="world" />
     <child link = "base_link" />
-    <origin xyz="0.0 0.0 0.0" rpy="0.0 0.0 0.0" />
+    <origin xyz="$(arg rob_xyz)" rpy="$(arg rob_rpy)" />
   </joint>
 </robot>
